Commit message: feat: prepare continuous AGV research demos and delivery evidence

File: src/my_bot_description/description/robot.urdf.xacro (robot description, xacro)
@@ -5,4 +5,7 @@
                      /scan va /odom do ESP32 phat, khong phai Gazebo. -->
     <xacro:arg name="sim" default="true" />
+    <!-- Fleet real: AGV1 blue, AGV2 orange. Defaults retain the simulation look. -->
+    <xacro:arg name="body_color" default="orange" />
+    <xacro:arg name="wheel_color" default="blue" />
     <!-- ====================================================================
          KICH THUOC XE
@@ -38,7 +41,7 @@
          robot_radius 0.13 (co bien 8 mm). -->
     <material name="white"><color rgba="1 1 1 1" /></material>
-    <material name="blue"><color rgba="0.2 0.2 1 1"/></material>
+    <material name="blue"><color rgba="0.15 0.45 0.95 1"/></material>
     <material name="black"><color rgba="0 0 0 1"/></material>
-    <material name="orange"><color rgba="1 0.5 0 1"/></material>
+    <material name="orange"><color rgba="0.95 0.5 0.1 1"/></material>
     <material name="red"><color rgba="1 0 0 1"/></material>
     <!-- base_footprint nam tren MAT SAN, ngay duoi TAM TRUC BANH (tam xoay cua xe
@@ -66,5 +69,5 @@
             <origin xyz="0 0 ${wheel_radius}"/>
             <geometry><cylinder radius="${body_radius}" length="${body_height}"/></geometry>
-            <material name="orange"/>
+            <material name="$(arg body_color)"/>
         </visual>
         <collision>
@@ -93,5 +96,5 @@
         <visual>
             <geometry><cylinder radius="${wheel_radius}" length="${wheel_width}"/></geometry>
-            <material name="blue"/>
+            <material name="$(arg wheel_color)"/>
         </visual>
         <collision>
@@ -118,5 +121,5 @@
         <visual>
             <geometry><cylinder radius="${wheel_radius}" length="${wheel_width}"/></geometry>
-            <material name="blue"/>
+            <material name="$(arg wheel_color)"/>
         </visual>
         <collision>
